Commit message: updated wip

File: ramsai_description/srdf/iiwa_macro.srdf.xacro (robot description, xacro)
@@ -2,15 +2,15 @@
 <robot xmlns:xacro="http://www.ros.org/wiki/xacro">
   <xacro:macro name="iiwa_print_srdf" params="name prefix">
-     <group name="${prefix}${name}_arm">
+     <group name="${prefix}iiwa_arm">
         <chain base_link="${prefix}iiwa_base" tip_link="${prefix}tool0" />
     </group>
-    <group_state name="ready" group="${prefix}${name}_arm">
-        <joint name="${prefix}joint_a1" value="0"/>
-        <joint name="${prefix}joint_a2" value="-0.785"/>
+    <group_state name="ready" group="${prefix}iiwa_arm">
+        <joint name="${prefix}joint_a1" value="-1.5707"/>
+        <joint name="${prefix}joint_a2" value="-0.7854"/>
         <joint name="${prefix}joint_a3" value="0"/>
-        <joint name="${prefix}joint_a4" value="-2.356"/>
+        <joint name="${prefix}joint_a4" value="1.3962"/>
         <joint name="${prefix}joint_a5" value="0"/>
-        <joint name="${prefix}joint_a6" value="1.571"/>
-        <joint name="${prefix}joint_a7" value="0.785"/>
+        <joint name="${prefix}joint_a6" value="0.6109"/>
+        <joint name="${prefix}joint_a7" value="0"/>
     </group_state>
     <virtual_joint child_link="${prefix}iiwa_base" name="virtual_joint" parent_frame="world" type="floating"/>
