Commit message: batch update curent work

File: ramsai_description/urdf/iiwa14.urdf.xacro (robot description, xacro)
@@ -190,5 +190,5 @@
         </collision>
     </link>
-    <link name="${prefix}lid" type="fixed">
+    <!-- <link name="${prefix}lid" type="fixed">
         <visual>
           <origin rpy="0 0 1.5708" xyz="0 0 0"/>
@@ -204,5 +204,5 @@
           </geometry>
         </collision>
-    </link>
+    </link> -->
     <link name="${prefix}flex_fellow" type="fixed">
         <visual>
@@ -276,16 +276,16 @@
         <axis xyz="0 0 0"/>
     </joint>
-    <joint name="${prefix}joint_a7-tool0" type="fixed">
-        <origin rpy="0 0 1.57" xyz="0.0 0.0 0.0"/> <!--0.154-->
+    <joint name="${prefix}extruder" type="fixed">
+        <origin rpy="0 0 -1.57" xyz="0.0 0.0 0.0"/> <!--0.154-->
         <parent link="${prefix}tip"/>
         <child link="${prefix}tool0"/>
         <axis xyz="0 0 0"/>
     </joint>
-    <joint name="${prefix}joint_base-lid" type="fixed">
+    <!-- <joint name="${prefix}joint_base-lid" type="fixed">
         <origin rpy="0 0.0 0" xyz="${Ox} ${Oy} ${Oz}"/>
         <parent link="${prefix}iiwa_base"/>
         <child link="${prefix}lid"/>
         <axis xyz="0 0 0"/>
-    </joint>
+    </joint> -->
     <joint name="${prefix}joint_base-flex" type="fixed">
         <origin rpy="0 0 0" xyz="0 0 0"/>
