Commit message: added hybrid planning config

File: ramsai_description/config/ramsai.config.xacro (robot description, xacro)
@@ -1,5 +1,5 @@
 <?xml version="1.0"?>
 <!-- Kuka iiwa 14 7DoF manipulator -->
-<robot xmlns:xacro="http://www.ros.org/wiki/xacro" name="iiwa14">
+<robot xmlns:xacro="http://www.ros.org/wiki/xacro" name="iiwa_print">
     <!-- Enable setting arguments from the launch file -->
     <xacro:arg name="use_sim" default="false" />
@@ -21,9 +21,9 @@
         <static>true</static>
     </gazebo>
-    <xacro:iiwa14 parent="world" prefix="$(arg prefix)">
+    <xacro:iiwa_print parent="world" prefix="$(arg prefix)">
         <origin xyz="0 0 0" rpy="0 0 0" />
-    </xacro:iiwa14>
+    </xacro:iiwa_print>
     <xacro:iiwa_r2c_hardware
-        name="iiwaRobot" prefix="$(arg prefix)"
+        name="iiwa_print" prefix="$(arg prefix)"
         robot_ip="$(arg robot_ip)" robot_port="$(arg robot_port)"
         command_interface="$(arg command_interface)"

File: ramsai_description/urdf/iiwa14.urdf.xacro (robot description, xacro)
@@ -1,290 +1,290 @@
 <?xml version="1.0"?>
 <robot xmlns:xacro="http://www.ros.org/wiki/xacro">
-  <xacro:macro name="iiwa14" params="parent prefix *origin">
-  <xacro:property name="Ox" value="0.0"/>
-  <xacro:property name="Oy" value="-0.75"/>
-  <xacro:property name="Oz" value="0.1"/>
-  <xacro:property name="dz" value="0.3259"/>
-  <xacro:property name="alpha" value="-0.6981"/>
-  <xacro:property name="l" value="0.0264"/>
-  <material name="gray">
-    <color rgba="0.5 0.5 0.5 1.0"/>
-  </material>
-  <link name="${prefix}iiwa_base" type="fixed"/>
-  <joint name="${prefix}iiwa_root_joint" type="fixed">
-      <xacro:insert_block name="origin" />
-      <parent link="${parent}"/>
-      <child link="${prefix}iiwa_base"/>
-  </joint>
-  <joint name="${prefix}iiwa_base_joint" type="fixed">
-      <origin rpy="0.0 0 0" xyz="0 0 0"/>
-      <parent link="${prefix}iiwa_base"/>
-      <child link="${prefix}link_0"/>
-  </joint>
-  <link name="${prefix}link_0">
-      <visual>
+  <xacro:macro name="iiwa_print" params="parent prefix *origin">
+    <xacro:property name="Ox" value="0.0"/>
+    <xacro:property name="Oy" value="-0.75"/>
+    <xacro:property name="Oz" value="0.1"/>
+    <xacro:property name="dz" value="0.3259"/>
+    <xacro:property name="alpha" value="-0.6981"/>
+    <xacro:property name="l" value="0.0264"/>
+    <material name="gray">
+      <color rgba="0.5 0.5 0.5 1.0"/>
+    </material>
+    <link name="${prefix}iiwa_base" type="fixed"/>
+    <joint name="${prefix}iiwa_root_joint" type="fixed">
+        <xacro:insert_block name="origin" />
+        <parent link="${parent}"/>
+        <child link="${prefix}iiwa_base"/>
+    </joint>
+    <joint name="${prefix}iiwa_base_joint" type="fixed">
         <origin rpy="0.0 0 0" xyz="0 0 0"/>
-        <geometry>
-          <mesh filename="package://iiwa_description/meshes/lbr_iiwa_14_r820/visual/base_link.dae"/>
-        </geometry>
-      </visual>
-      <collision>
-        <origin rpy="0 0 0" xyz="0 0 0"/>
-        <geometry>
-          <mesh filename="package://iiwa_description/meshes/lbr_iiwa_14_r820/collision/base_link.stl"/>
-        </geometry>
-      </collision>
-      <inertial>
-        <origin xyz="-0.1 0 0.07" rpy="0 0 0"/>
-        <mass value="5"/>
-        <inertia ixx="0.05"  ixy="0"  ixz="0" iyy="0.06" iyz="0" izz="0.03" />
-      </inertial>
-  </link>
-  <link name="${prefix}link_1">
-      <visual>
-        <origin rpy="0 0 0" xyz="0 0 0"/>
-        <geometry>
-          <mesh filename="package://iiwa_description/meshes/lbr_iiwa_14_r820/visual/link_1.dae"/>
-        </geometry>
-      </visual>
-      <collision>
-        <origin rpy="0 0 0" xyz="0 0 0"/>
-        <geometry>
-          <mesh filename="package://iiwa_description/meshes/lbr_iiwa_14_r820/collision/link_1.stl"/>
-        </geometry>
-      </collision>
-      <inertial>
-        <origin xyz="0 -0.03 0.12" rpy="0 0 0"/>
-        <mass value="4"/>
-        <inertia ixx="0.1"  ixy="0"  ixz="0" iyy="0.09" iyz="0" izz="0.02" />
-      </inertial>
-  </link>
-  <link name="${prefix}link_2">
-      <visual>
-        <origin rpy="0 0 0" xyz="0 0 0"/>
-        <geometry>
-          <mesh filename="package://iiwa_description/meshes/lbr_iiwa_14_r820/visual/link_2.dae"/>
-        </geometry>
-      </visual>
-      <collision>
-        <origin rpy="0 0 0" xyz="0 0 0"/>
-        <geometry>
-          <mesh filename="package://iiwa_description/meshes/lbr_iiwa_14_r820/collision/link_2.stl"/>
-        </geometry>
-      </collision>
-      <inertial>
-        <origin xyz="0.0003 0.059 0.042" rpy="0 0 0"/>
-        <mass value="4"/>
-        <inertia ixx="0.05"  ixy="0"  ixz="0" iyy="0.018" iyz="0" izz="0.044" />
-      </inertial>
-  </link>
-  <link name="${prefix}link_3">
-      <visual>
-        <origin rpy="0 0 0" xyz="0 0 0"/>
-        <geometry>
-          <mesh filename="package://iiwa_description/meshes/lbr_iiwa_14_r820/visual/link_3.dae"/>
-        </geometry>
-      </visual>
-      <collision>
-        <origin rpy="0 0 0" xyz="0 0 0"/>
-        <geometry>
-          <mesh filename="package://iiwa_description/meshes/lbr_iiwa_14_r820/collision/link_3.stl"/>
-        </geometry>
-      </collision>
-      <inertial>
-        <origin xyz="0 0.03 0.13" rpy="0 0 0"/>
-        <mass value="3"/>
-        <inertia ixx="0.08"  ixy="0"  ixz="0" iyy="0.075" iyz="0" izz="0.01" />
-      </inertial>
-  </link>
-  <link name="${prefix}link_4">
-      <visual>
-        <origin rpy="0 0 0" xyz="0 0 0"/>
-        <geometry>
-          <mesh filename="package://iiwa_description/meshes/lbr_iiwa_14_r820/visual/link_4.dae"/>
-        </geometry>
-      </visual>
-      <collision>
-        <origin rpy="0 0 0" xyz="0 0 0"/>
-        <geometry>
-          <mesh filename="package://iiwa_description/meshes/lbr_iiwa_14_r820/collision/link_4.stl"/>
-        </geometry>
-      </collision>
-      <inertial>
-        <origin xyz="0 0.067 0.034" rpy="0 0 0"/>
-        <mass value="2.7"/>
-        <inertia ixx="0.03"  ixy="0"  ixz="0" iyy="0.01" iyz="0" izz="0.029" />
-      </inertial>
-  </link>
-  <link name="${prefix}link_5">
-      <visual>
-        <origin rpy="0 0 0" xyz="0 0 0"/>
-        <geometry>
-          <mesh filename="package://iiwa_description/meshes/lbr_iiwa_14_r820/visual/link_5.dae"/>
-        </geometry>
-      </visual>
-      <collision>
-        <origin rpy="0 0 0" xyz="0 0 0"/>
-        <geometry>
-          <mesh filename="package://iiwa_description/meshes/lbr_iiwa_14_r820/collision/link_5.stl"/>
-        </geometry>
-      </collision>
-      <inertial>
-        <origin xyz="0.0001 0.021 0.076" rpy="0 0 0"/>
-        <mass value="1.7"/>
-        <inertia ixx="0.02"  ixy="0"  ixz="0" iyy="0.018" iyz="0" izz="0.005" />
-      </inertial>
-  </link>
-  <link name="${prefix}link_6">
-      <visual>
-        <origin rpy="0 0 0" xyz="0 0 0"/>
-        <geometry>
-          <mesh filename="package://iiwa_description/meshes/lbr_iiwa_14_r820/visual/link_6.dae"/>
-        </geometry>
-      </visual>
-      <collision>
-        <origin rpy="0 0 0" xyz="0 0 0"/>
-        <geometry>
-          <mesh filename="package://iiwa_description/meshes/lbr_iiwa_14_r820/collision/link_6.stl"/>
-        </geometry>
-      </collision>
-      <inertial>
-        <origin xyz="0 0.0006 0.0004" rpy="0 0 0"/>
-        <mass value="1.8"/>
-        <inertia ixx="0.025"  ixy="0"  ixz="0" iyy="0.0136" iyz="0" izz="0.0247" />
-      </inertial>
-  </link>
-  <link name="${prefix}link_7">
-      <visual>
-        <origin rpy="0 0 0" xyz="0 0 0.07"/>
-        <material name="gray"/>
-        <geometry>
-          <mesh filename="package://ramsai_description/meshes/viscotec/visual/link_7_2.stl" scale ="0.001 0.001 0.001"/>
-        </geometry>
-      </visual>
-      <collision>
-        <origin rpy="0 0 0" xyz="0 0 0.07"/>
-        <geometry>
-          <mesh filename="package://ramsai_description/meshes/viscotec/collision/link_7_2.stl" scale ="0.001 0.001 0.001"/>
-        </geometry>
-      </collision>
-      <inertial>
-        <origin xyz="0 0 0.02" rpy="0 0 0"/>
-        <mass value="${0.3 / 0.308 * 0.44}"/> <!--this is for the MFT Pneumatisch flange-->
-        <inertia ixx="0.01"  ixy="0"  ixz="0" iyy="0.01" iyz="0" izz="0.01" />
-      </inertial>
-  </link>
-  <link name="${prefix}tool0">
-      <visual>
-        <origin rpy="0 ${-alpha} 0" xyz="-0.1118 0 -0.1333"/>
-        <material name="gray"/>
-        <geometry>
-          <mesh filename="package://ramsai_description/meshes/viscotec/visual/viscotec.dae" scale ="0.001 0.001 0.001"/>
-        </geometry>
-      </visual>
-      <collision>
-        <origin rpy="0 ${-alpha} 0" xyz="-0.1118 0 -0.1333"/>
-        <geometry>
-          <mesh filename="package://ramsai_description/meshes/viscotec/collision/viscotec.stl" scale ="0.001 0.001 0.001"/>
-        </geometry>
-      </collision>
-  </link>
-  <link name="${prefix}lid" type="fixed">
-      <visual>
-        <origin rpy="0 0 1.5708" xyz="0 0 0"/>
-        <material name="gray"/>
-        <geometry>
-          <mesh filename="package://ramsai_description/meshes/viscotec/visual/cell.dae" scale ="0.001 0.001 0.001"/>
-        </geometry>
-      </visual>
-      <collision>
-        <origin rpy="0 0 1.5708" xyz="0 0 0"/>
-        <geometry>
-          <mesh filename="package://ramsai_description/meshes/viscotec/collision/cell.stl" scale ="0.001 0.001 0.001"/>
-        </geometry>
-      </collision>
-  </link>
-  <link name="${prefix}flex_fellow" type="fixed">
-      <visual>
-        <origin rpy="3.1415 0 3.1415" xyz="0 0 0"/>
-        <material name="gray"/>
-        <geometry>
-          <mesh filename="package://ramsai_description/meshes/flex_fellow_h800/flex_fellow_h800.dae" scale ="1 1 1"/>
-        </geometry>
-      </visual>
-      <collision>
-        <origin rpy="3.1415 0 1.5708" xyz="0 0 0"/>
-        <geometry>
-          <mesh filename="package://ramsai_description/meshes/flex_fellow_h800/flex_fellow_h800.stl" scale ="1 1 1"/>
-        </geometry>
-      </collision>
-  </link>
-  <joint name="${prefix}joint_a1" type="revolute">
-      <origin rpy="0 0 0" xyz="0 0 0"/>
-      <parent link="${prefix}link_0"/>
-      <child link="${prefix}link_1"/>
-      <axis xyz="0 0 1"/>
-      <limit effort="320" lower="-2.9668" upper="2.9668" velocity="1.4834"/>
-  </joint>
-  <joint name="${prefix}joint_a2" type="revolute">
-      <origin rpy="0 0 0" xyz="-0.00043624 0 0.36"/>
-      <parent link="${prefix}link_1"/>
-      <child link="${prefix}link_2"/>
-      <axis xyz="0 1 0"/>
-      <limit effort="320" lower="-2.0942" upper="2.0942" velocity="1.4834"/>
-  </joint>
-  <joint name="${prefix}joint_a3" type="revolute">
-      <origin rpy="0 0 0" xyz="0 0 0"/>
-      <parent link="${prefix}link_2"/>
-      <child link="${prefix}link_3"/>
-      <axis xyz="0 0 1"/>
-      <limit effort="176" lower="-2.9668" upper="2.9668" velocity="1.7452"/>
-  </joint>
-  <joint name="${prefix}joint_a4" type="revolute">
-      <origin rpy="0 0 0" xyz="0.00043624 0 0.42"/>
-      <parent link="${prefix}link_3"/>
-      <child link="${prefix}link_4"/>
-      <axis xyz="0 -1 0"/>
-      <limit effort="176" lower="-2.0942" upper="2.0942" velocity="1.3089"/>
-  </joint>
-  <joint name="${prefix}joint_a5" type="revolute">
-      <origin rpy="0 0 0" xyz="0 0 0"/>
-      <parent link="${prefix}link_4"/>
-      <child link="${prefix}link_5"/>
-      <axis xyz="0 0 1"/>
-      <limit effort="110" lower="-2.9668" upper="2.9668" velocity="2.2688"/>
-  </joint>
-  <joint name="${prefix}joint_a6" type="revolute">
-      <origin rpy="0 0 0" xyz="0 0 0.4"/>
-      <parent link="${prefix}link_5"/>
-      <child link="${prefix}link_6"/>
-      <axis xyz="0 1 0"/>
-      <limit effort="40" lower="-2.0942" upper="2.0942" velocity="2.356"/>
-  </joint>
-  <joint name="${prefix}joint_a7" type="revolute">
-      <origin rpy="0 0 0" xyz="0 0 0"/>
-      <parent link="${prefix}link_6"/>
-      <child link="${prefix}link_7"/>
-      <axis xyz="0 0 1"/>
-      <limit effort="40" lower="-3.0541" upper="3.0541" velocity="2.356"/>
-  </joint>
-  <joint name="${prefix}joint_a7-tool0" type="fixed">
-      <origin rpy="0 ${alpha} 0" xyz="${sin(alpha)*(l-0.0264)} 0.0 ${dz+cos(alpha)*(l-0.0264)}"/> <!--0.154-->
-      <parent link="${prefix}link_7"/>
-      <child link="${prefix}tool0"/>
-      <axis xyz="0 0 0"/>
-  </joint>
-  <joint name="${prefix}joint_base-lid" type="fixed">
-      <origin rpy="0 0.0 0" xyz="${Ox} ${Oy} ${Oz}"/>
-      <parent link="${prefix}iiwa_base"/>
-      <child link="${prefix}lid"/>
-      <axis xyz="0 0 0"/>
-  </joint>
-  <joint name="${prefix}joint_base-flex" type="fixed">
-      <origin rpy="0 0 0" xyz="0 0 0"/>
-      <parent link="${prefix}iiwa_base"/>
-      <child link="${prefix}flex_fellow"/>
-      <axis xyz="0 0 0"/>
-  </joint>
+        <parent link="${prefix}iiwa_base"/>
+        <child link="${prefix}link_0"/>
+    </joint>
+    <link name="${prefix}link_0">
+        <visual>
+          <origin rpy="0.0 0 0" xyz="0 0 0"/>
+          <geometry>
+            <mesh filename="package://iiwa_description/meshes/lbr_iiwa_14_r820/visual/base_link.dae"/>
+          </geometry>
+        </visual>
+        <collision>
+          <origin rpy="0 0 0" xyz="0 0 0"/>
+          <geometry>
+            <mesh filename="package://iiwa_description/meshes/lbr_iiwa_14_r820/collision/base_link.stl"/>
+          </geometry>
+        </collision>
+        <inertial>
+          <origin xyz="-0.1 0 0.07" rpy="0 0 0"/>
+          <mass value="5"/>
+          <inertia ixx="0.05"  ixy="0"  ixz="0" iyy="0.06" iyz="0" izz="0.03" />
+        </inertial>
+    </link>
+    <link name="${prefix}link_1">
+        <visual>
+          <origin rpy="0 0 0" xyz="0 0 0"/>
+          <geometry>
+            <mesh filename="package://iiwa_description/meshes/lbr_iiwa_14_r820/visual/link_1.dae"/>
+          </geometry>
+        </visual>
+        <collision>
+          <origin rpy="0 0 0" xyz="0 0 0"/>
+          <geometry>
+            <mesh filename="package://iiwa_description/meshes/lbr_iiwa_14_r820/collision/link_1.stl"/>
+          </geometry>
+        </collision>
+        <inertial>
+          <origin xyz="0 -0.03 0.12" rpy="0 0 0"/>
+          <mass value="4"/>
+          <inertia ixx="0.1"  ixy="0"  ixz="0" iyy="0.09" iyz="0" izz="0.02" />
+        </inertial>
+    </link>
+    <link name="${prefix}link_2">
+        <visual>
+          <origin rpy="0 0 0" xyz="0 0 0"/>
+          <geometry>
+            <mesh filename="package://iiwa_description/meshes/lbr_iiwa_14_r820/visual/link_2.dae"/>
+          </geometry>
+        </visual>
+        <collision>
+          <origin rpy="0 0 0" xyz="0 0 0"/>
+          <geometry>
+            <mesh filename="package://iiwa_description/meshes/lbr_iiwa_14_r820/collision/link_2.stl"/>
+          </geometry>
+        </collision>
+        <inertial>
+          <origin xyz="0.0003 0.059 0.042" rpy="0 0 0"/>
+          <mass value="4"/>
+          <inertia ixx="0.05"  ixy="0"  ixz="0" iyy="0.018" iyz="0" izz="0.044" />
+        </inertial>
+    </link>
+    <link name="${prefix}link_3">
+        <visual>
+          <origin rpy="0 0 0" xyz="0 0 0"/>
+          <geometry>
+            <mesh filename="package://iiwa_description/meshes/lbr_iiwa_14_r820/visual/link_3.dae"/>
+          </geometry>
+        </visual>
+        <collision>
+          <origin rpy="0 0 0" xyz="0 0 0"/>
+          <geometry>
+            <mesh filename="package://iiwa_description/meshes/lbr_iiwa_14_r820/collision/link_3.stl"/>
+          </geometry>
+        </collision>
+        <inertial>
+          <origin xyz="0 0.03 0.13" rpy="0 0 0"/>
+          <mass value="3"/>
+          <inertia ixx="0.08"  ixy="0"  ixz="0" iyy="0.075" iyz="0" izz="0.01" />
+        </inertial>
+    </link>
+    <link name="${prefix}link_4">
+        <visual>
+          <origin rpy="0 0 0" xyz="0 0 0"/>
+          <geometry>
+            <mesh filename="package://iiwa_description/meshes/lbr_iiwa_14_r820/visual/link_4.dae"/>
+          </geometry>
+        </visual>
+        <collision>
+          <origin rpy="0 0 0" xyz="0 0 0"/>
+          <geometry>
+            <mesh filename="package://iiwa_description/meshes/lbr_iiwa_14_r820/collision/link_4.stl"/>
+          </geometry>
+        </collision>
+        <inertial>
+          <origin xyz="0 0.067 0.034" rpy="0 0 0"/>
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
Commit message: fixed merge

File: ramsai_description/config/ramsai.config.xacro (robot description, xacro)
@@ -14,4 +14,6 @@
     <!-- Import iiwa ros2_control description -->
     <xacro:include filename="$(find iiwa_description)/ros2_control/iiwa.r2c_hardware.xacro" />
+    <!-- Import extruder ros2_control description -->
+    <xacro:include filename="$(find ramsai_description)/ros2_control/extruder.ros2_control.xacro" />
     <!-- Import all Gazebo-customization elements -->
     <!-- <xacro:include filename="$(find iiwa_description)/gazebo/iiwa.gazebo"/> -->
@@ -31,3 +33,4 @@
         use_sim="$(arg use_sim)" use_fake_hardware="$(arg use_fake_hardware)"
         />
+    <xacro:extruder/>
 </robot>

File: ramsai_description/urdf/iiwa14.urdf.xacro (robot description, xacro)
@@ -175,5 +175,5 @@
         </inertial>
     </link>
-    <link name="${prefix}tool0">
+    <link name="${prefix}tip">
         <visual>
           <origin rpy="0 ${-alpha} 0" xyz="-0.1118 0 -0.1333"/>
@@ -220,4 +220,5 @@
         </collision>
     </link>
+    <link name="${prefix}tool0"/>
     <joint name="${prefix}joint_a1" type="revolute">
         <origin rpy="0 0 0" xyz="0 0 0"/>
@@ -269,7 +270,13 @@
         <limit effort="40" lower="-3.0541" upper="3.0541" velocity="2.356"/>
     </joint>
-    <joint name="${prefix}joint_a7-tool0" type="fixed">
+    <joint name="${prefix}joint_a7-tip" type="fixed">
         <origin rpy="0 ${alpha} 0" xyz="${sin(alpha)*(l-0.0264)} 0.0 ${dz+cos(alpha)*(l-0.0264)}"/> <!--0.154-->
         <parent link="${prefix}link_7"/>
+        <child link="${prefix}tip"/>
+        <axis xyz="0 0 0"/>
+    </joint>
+    <joint name="${prefix}joint_a7-tool0" type="fixed">
+        <origin rpy="0 0 1.57" xyz="0.0 0.0 0.0"/> <!--0.154-->
+        <parent link="${prefix}tip"/>
         <child link="${prefix}tool0"/>
         <axis xyz="0 0 0"/>

Commit message: Working set up

File: ramsai_description/config/ramsai.config.xacro (robot description, xacro)
@@ -33,4 +33,4 @@
         use_sim="$(arg use_sim)" use_fake_hardware="$(arg use_fake_hardware)"
         />
-    <xacro:extruder/>
+<!--    <xacro:extruder/> -->
 </robot>

File: ramsai_description/ros2_control/extruder.ros2_control.xacro (robot description, xacro)
@@ -1,10 +1,14 @@
 <?xml version="1.0"?>
 <robot xmlns:xacro="http://www.ros.org/wiki/xacro">
-  <xacro:macro name="extruder">
+  <xacro:macro
+    name="r2c_extruder"
+    params="use_fake_hardware">
     <ros2_control name="extruder" type="system">
       <hardware>
-        <plugin>ethercat_driver/EthercatDriver</plugin>
-        <param name="master_id">0</param>
-        <param name="control_frequency">225</param>
+        <xacro:unless value="{$use_fake_hardware}">
+          <plugin>ethercat_driver/EthercatDriver</plugin>
+          <param name="master_id">0</param>
+          <param name="control_frequency">225</param>
+        </xacro:unless>
       </hardware>
       <joint name="extruder">
@@ -19,10 +23,12 @@
         <command_interface name="reset"/>
         <command_interface name="velocity"/>
-        <ec_module name="viprohead">
-          <plugin>ethercat_generic_plugins/GenericEcSlave</plugin>
-          <param name="alias">0</param>
-          <param name="position">1</param>
-          <param name="slave_config">$(find ramsai_description)/config/bhf_el7031_config.yaml</param>
-        </ec_module>
+        <xacro:unless value="${use_fake_hardware}">
+          <ec_module name="viprohead">
+            <plugin>ethercat_generic_plugins/GenericEcSlave</plugin>
+            <param name="alias">0</param>
+            <param name="position">1</param>
+            <param name="slave_config">$(find ramsai_description)/config/bhf_el7031_config.yaml</param>
+          </ec_module>
+         </xacro:unless>
       </joint>
     </ros2_control>

File: ramsai_description/urdf/iiwa14.urdf.xacro (robot description, xacro)
@@ -175,5 +175,5 @@
         </inertial>
     </link>
-    <link name="${prefix}tip">
+    <link name="${prefix}tool0">
         <visual>
           <origin rpy="0 ${-alpha} 0" xyz="-0.1118 0 -0.1333"/>
@@ -220,5 +220,4 @@
         </collision>
     </link>
-    <link name="${prefix}tool0"/>
     <joint name="${prefix}joint_a1" type="revolute">
         <origin rpy="0 0 0" xyz="0 0 0"/>
@@ -270,17 +269,17 @@
         <limit effort="40" lower="-3.0541" upper="3.0541" velocity="2.356"/>
     </joint>
-    <joint name="${prefix}joint_a7-tip" type="fixed">
-        <origin rpy="0 ${alpha} 0" xyz="${sin(alpha)*(l-0.0264)} 0.0 ${dz+cos(alpha)*(l-0.0264)}"/> <!--0.154-->
+    <joint name="${prefix}joint_a7-tool0" type="fixed">
+        <origin rpy="0 ${alpha} 3.14" xyz="${sin(alpha)*(l-0.0264)} 0.0 ${dz+cos(alpha)*(l-0.0264)}"/> <!--0.154-->
         <parent link="${prefix}link_7"/>
-        <child link="${prefix}tip"/>
-        <axis xyz="0 0 0"/>
-    </joint>
-    <joint name="${prefix}extruder" type="fixed">
-        <origin rpy="0 0 -1.57" xyz="0.0 0.0 0.0"/> <!--0.154-->
+        <child link="${prefix}tool0"/>
+        <axis xyz="0 0 0"/>
+    </joint>
+  <!--  <joint name="${prefix}extruder" type="fixed">
+        <origin rpy="0 0 -1.57" xyz="0.0 0.0 0.0"/> <!-0.154->
         <parent link="${prefix}tip"/>
         <child link="${prefix}tool0"/>
         <axis xyz="0 0 0"/>
-    </joint>
-    <!-- <joint name="${prefix}joint_base-lid" type="fixed">
+    </joint> -->
+  <!--<joint name="${prefix}joint_base-lid" type="fixed">
         <origin rpy="0 0.0 0" xyz="${Ox} ${Oy} ${Oz}"/>
         <parent link="${prefix}iiwa_base"/>
